Commit message: Added apartment scene with working simulated sensors

File: src/control_hardware/urdf/ignition_ros2_control.xacro (robot description, xacro)
@@ -8,11 +8,13 @@
       <command_interface name="velocity" />
       <state_interface name="velocity" />
+      <state_interface name="position" />
     </joint>
     <joint name="Revolute_Right_Wheel">
       <command_interface name="velocity" />
       <state_interface name="velocity" />
+      <state_interface name="position" />
     </joint>
   </ros2_control>
-    <!-- Gazebo's ros2_control plugin -->
+  <!-- Gazebo's ros2_control plugin -->
   <gazebo>
     <plugin filename="libign_ros2_control-system.so" name="ign_ros2_control::IgnitionROS2ControlPlugin">

File: src/control_hardware/urdf/real_ros2_control.xacro (robot description, xacro)
@@ -21,5 +21,5 @@
     <hardware>
       <plugin>control_hardware/DM542_Stepper_ActuatorHardware</plugin>
-      <param name="pul_pin">12</param>
+      <param name="pul_pin">23</param>
       <param name="en_pin">27</param>
       <param name="dir_pin">22</param>

File: src/control_hardware/urdf/sim_snack_robot.xacro (robot description, xacro)
@@ -3,3 +3,4 @@
   <xacro:include filename="$(find robot_model_export_description)/urdf/robot_model_export.xacro" />
   <xacro:include filename="$(find control_hardware)/urdf/ignition_ros2_control.xacro" />
+  <xacro:include filename="$(find control_hardware)/urdf/ign_sensors.xacro" />
 </robot>

File: src/robot_model_export_description/urdf/robot_model_export.xacro (robot description, xacro)
@@ -48,5 +48,5 @@
     <origin xyz="3.243495146770803e-08 -0.005407956920820883 3.930996579964291e-05" rpy="0 0 0"/>
     <mass value="0.006547683530071288"/>
-    <inertia ixx="1e-06" iyy="0.0" izz="1e-06" ixy="-0.0" iyz="0.0" ixz="0.0"/>
+    <inertia ixx="1e-06" iyy="1e-06" izz="1e-06" ixy="-0.0" iyz="0.0" ixz="0.0"/>
   </inertial>
   <visual>
@@ -140,5 +140,5 @@
     <origin xyz="3.2434951495463604e-08 0.005408386207586657 3.930996579963597e-05" rpy="0 0 0"/>
     <mass value="0.00654768353007129"/>
-    <inertia ixx="1e-06" iyy="0.0" izz="1e-06" ixy="0.0" iyz="-0.0" ixz="0.0"/>
+    <inertia ixx="1e-06" iyy="1e-06" izz="1e-06" ixy="0.0" iyz="-0.0" ixz="0.0"/>
   </inertial>
   <visual>
@@ -466,5 +466,5 @@
   <parent link="Right_Motor_Mirror___1__1"/>
   <child link="Right_Wheel_Attachment_Mirror__1"/>
-  <axis xyz="-0.0 -1.0 0.0"/>
+  <axis xyz="0.0 -1.0 0.0"/>
 </joint>
 <joint name="Rigid 22" type="fixed">
