Commit message: Fixed a bunch of bugs, found more

File: src/control_hardware/urdf/real_ros2_control.xacro (robot description, xacro)
@@ -26,5 +26,5 @@
       <param name="pulse_per_rev">1600</param>
     </hardware>
-    <joint name="Left_Wheel_Actuator">
+    <joint name="Revolute_Left_Wheel">
       <state_interface name="position" />
       <state_interface name="velocity" />
@@ -40,5 +40,5 @@
       <param name="pulse_per_rev">1600</param>
     </hardware>
-    <joint name="Right_Wheel_Actuator">
+    <joint name="Revolute_Right_Wheel">
       <state_interface name="position" />
       <state_interface name="velocity" />

File: src/robot_model_export_description/urdf/robot_model_export.xacro (robot description, xacro)
@@ -176,5 +176,5 @@
   </collision>
 </link>
-<link name="IMU_1">
+<link name="imu_link">
   <inertial>
     <origin xyz="0.008109521073689362 2.1464338289019908e-07 0.0010279143883868743" rpy="0 0 0"/>
@@ -473,8 +473,8 @@
   <child link="Right_Wheel_Mirror__1"/>
 </joint>
-<joint name="imu_link" type="fixed">
+<joint name="IMU" type="fixed">
   <origin xyz="-0.05822 3.5e-05 0.00813" rpy="0 0 0"/>
   <parent link="base_link"/>
-  <child link="IMU_1"/>
+  <child link="imu_link"/>
 </joint>
 <joint name="Rigid 24" type="fixed">

Commit message: Changed motor implementation to use dynamixel motors since stepper straight up didn't work

File: src/control_hardware/urdf/real_ros2_control.xacro (robot description, xacro)
@@ -18,33 +18,49 @@
     </sensor>
   </ros2_control>
-  <ros2_control name="LeftStepper" type="actuator" rw_rate="50">
+  <ros2_control name="LeftStepper" type="system" rw_rate="50">
     <hardware>
-      <plugin>control_hardware/DM542_Stepper_ActuatorHardware</plugin>
-      <param name="pul_pin">23</param>
-      <param name="en_pin">27</param>
-      <param name="dir_pin">22</param>
-      <param name="pulse_per_rev">1600</param>
-      <param name="direction_multiplier">1.0</param>
+      <plugin>dynamixel_hardware_interface/DynamixelHardware</plugin>
+      <param name="port_name">/dev/USB0</param>
+      <param name="baud_rate">9600</param>
+      <param name="error_timeout_ms">100</param>
+      <param name="number_of_joints">2</param>
+      <param name="number_of_transmissions">0</param>
     </hardware>
     <joint name="Revolute_Left_Wheel">
+      <command_interface name="velocity" />
       <state_interface name="position" />
       <state_interface name="velocity" />
+      <state_interface name="effort" />
+    </joint>
+    <joint name="Revolute_Right_Wheel">
       <command_interface name="velocity" />
-    </joint>
-  </ros2_control>
-  <ros2_control name="RightStepper" type="actuator" rw_rate="50">
-    <hardware>
-      <plugin>control_hardware/DM542_Stepper_ActuatorHardware</plugin>
-      <param name="pul_pin">13</param>
-      <param name="en_pin">5</param>
-      <param name="dir_pin">6</param>
-      <param name="pulse_per_rev">1600</param>
-      <param name="direction_multiplier">-1.0</param>
-    </hardware>
-    <joint name="Revolute_Right_Wheel">
       <state_interface name="position" />
       <state_interface name="velocity" />
-      <command_interface name="velocity" />
+      <state_interface name="effort" />
     </joint>
+    <gpio name="left_wheel">
+      <param name="type">dxl</param>
+      <param name="ID">11</param>
+      <command_interface name="Goal Velocity" />
+      <state_interface name="Present Position"/>
+      <state_interface name="Present Velocity"/>
+      <state_interface name="Present Current"/>
+      <param name="Position P Gain">800</param> <!-- Proportional gain for position control -->
+      <param name="Position I Gain">100</param> <!-- Integral gain for position control -->
+      <param name="Position D Gain">100</param> <!-- Derivative gain for position control -->
+      <param name="Drive Mode">0</param> <!-- 0: Clockwise, 1: Counterclockwise -->
+    </gpio>
+    <gpio name="right_wheel">
+      <param name="type">dxl</param>
+      <param name="ID">12</param>
+      <command_interface name="Goal Velocity" />
+      <state_interface name="Present Position"/>
+      <state_interface name="Present Velocity"/>
+      <state_interface name="Present Current"/>
+      <param name="Position P Gain">800</param> <!-- Proportional gain for position control -->
+      <param name="Position I Gain">100</param> <!-- Integral gain for position control -->
+      <param name="Position D Gain">100</param> <!-- Derivative gain for position control -->
+      <param name="Drive Mode">1</param> <!-- 0: Clockwise, 1: Counterclockwise -->
+    </gpio>
   </ros2_control>
     <!-- Gazebo's ros2_control plugin -->
